File: grbl_board/power_supply.sch (KiCad schematic (older format))
At the start: 0 parts

Commit message: power supply stage
Parts:
- added C? (x2): 470u, symbol Device:C
- added C? (x3): 10u, symbol Device:C
- added C?: 100n, symbol Device:C
- added C?: 6.8n, symbol Device:C
- added C?: 100u, symbol Device:C
- added C?: 1u, symbol Device:C
- added C?: 10n, symbol Device:C
- added D?: SS2150-LTP, symbol Device:D_Schottky
- added F?: 2A, symbol Device:Polyfuse
- added F?: 300mA, symbol Device:Polyfuse
- added J?: 32VDC, symbol Connector:Screw_Terminal_01x02
- added L?: 20u, symbol Device:L
- added L?: 33u, symbol Device:L
- added R? (x2): 1, symbol Device:R
- added R?: 47k, symbol Device:R
- added R?: 10k, symbol Device:R
- added R?: 2.2k, symbol Device:R
- added R?: 200, symbol Device:R
- added U?: BD9G341EFJ, Package_SO:HTSOP-8-1EP_3.9x4.9mm_P1.27mm_EP2.4x3.2mm_ThermalVias, symbol Regulator_Switching:BD9G341EFJ
- added U?: LT1962-5, Package_SO:MSOP-8_3x3mm_P0.65mm, symbol Regulator_Linear:LT1962-5
Connections:
- new net: D?.1 (K), L?.1, U?.1 (LX), U?.7 (BST)
- new net: C?.1, U?.3 (VC)
- new net: R?.1, R?.2, U?.4 (FB)
- new net: R?.1, U?.5 (RT)
- new net: R?.1, R?.2, U?.6 (EN)
- new net: C?.1, J?.2 (Pin_2), L?.1
- new net: C?.2, R?.1
- new net: C?.1, F?.2, L?.2, R?.1
- new net: C?.1, C?.1, F?.2, U?.1 (OUT), U?.2 (SENSE)
- new net: C?.2, U?.3 (BYP)
- new net 12VDC: C?.1, F?.1, U?.5 (~SHDN), U?.8 (IN)
- new net 32VDC: C?.1, C?.1, C?.1, C?.1, L?.2, R?.1, U?.8 (VCC)
- new net 5VDC: F?.1
- new net GND: C?.2, C?.2, C?.2, C?.2, C?.2, C?.2, C?.2, C?.2, D?.2 (A), J?.1 (Pin_1), R?.2, R?.2, R?.2, R?.2, U?.2 (GND), U?.4 (GND)
