File: grbl_board/stepper_drivers.sch (KiCad schematic (older format))
At the start: 0 parts

Commit message: motor driver and mcu and limit switches
Parts:
- added D? (x36): B360, Diode_SMD:D_SMC, symbol Diode:B360
- added J?: X_STEPPER, symbol Connector:Screw_Terminal_01x04
- added J?: Y_STEPPER, symbol Connector:Screw_Terminal_01x04
- added J?: Z_STEPPER, symbol Connector:Screw_Terminal_01x04
- added J?: E_STEPPER, symbol Connector:Screw_Terminal_01x04
- added U? (x4): TMC5160_SILENTSTEPSTICK, grbl_board:TMC5160_SILENTSTEPSTICK, symbol grbl_board:TMC5160_SILENTSTEPSTICK
Connections:
- new net: D?.1 (K), D?.2 (A), J?.1 (Pin_1), U?.JP2_3 (OA2) (x4)
- new net: D?.1 (K), D?.2 (A), J?.2 (Pin_2), U?.JP2_4 (OA1) (x4)
- new net: D?.1 (K), D?.2 (A), J?.3 (Pin_3), U?.JP2_5 (OB1) (x4)
- new net: D?.1 (K), D?.2 (A), J?.4 (Pin_4), U?.JP2_6 (OB2) (x4)
- new net: D?.2 (A), U?.JP2_7 (VIO) (x4)
- new net CS_E: U?.JP1_5 (CSN)
- new net CS_X: U?.JP1_5 (CSN)
- new net CS_Y: U?.JP1_5 (CSN)
- new net CS_Z: U?.JP1_5 (CSN)
- new net EN: U?.JP1_8 (EN), U?.JP1_8 (EN), U?.JP1_8 (EN), U?.JP1_8 (EN)
- new net E_DIR: U?.JP1_1 (DIR)
- new net E_STEP: U?.JP1_2 (STEP)
- new net GND: D?.2 (A), D?.2 (A), D?.2 (A), D?.2 (A), D?.2 (A), D?.2 (A), D?.2 (A), D?.2 (A), D?.2 (A), D?.2 (A), D?.2 (A), D?.2 (A), D?.2 (A), D?.2 (A), D?.2 (A), D?.2 (A), U?.JP1_3 (CLK), U?.JP1_3 (CLK), U?.JP1_3 (CLK), U?.JP1_3 (CLK), U?.JP2_2 (GND), U?.JP2_2 (GND), U?.JP2_2 (GND), U?.JP2_2 (GND), U?.JP2_8 (GND), U?.JP2_8 (GND), U?.JP2_8 (GND), U?.JP2_8 (GND)
- new net MISO: U?.JP1_4 (SDO), U?.JP1_4 (SDO), U?.JP1_4 (SDO), U?.JP1_4 (SDO)
- new net MOSI: U?.JP1_7 (SDI), U?.JP1_7 (SDI), U?.JP1_7 (SDI), U?.JP1_7 (SDI)
- new net SCK: U?.JP1_6 (SCK), U?.JP1_6 (SCK), U?.JP1_6 (SCK), U?.JP1_6 (SCK)
- new net VMOT: D?.1 (K), D?.1 (K), D?.1 (K), D?.1 (K), D?.1 (K), D?.1 (K), D?.1 (K), D?.1 (K), D?.1 (K), D?.1 (K), D?.1 (K), D?.1 (K), D?.1 (K), D?.1 (K), D?.1 (K), D?.1 (K), D?.1 (K), D?.1 (K), D?.1 (K), D?.1 (K), U?.JP2_1 (VM), U?.JP2_1 (VM), U?.JP2_1 (VM), U?.JP2_1 (VM)
- new net X_DIR: U?.JP1_1 (DIR)
- new net X_STEP: U?.JP1_2 (STEP)
- new net Y_DIR: U?.JP1_1 (DIR)
- new net Y_STEP: U?.JP1_2 (STEP)
- new net Z_DIR: U?.JP1_1 (DIR)
- new net Z_STEP: U?.JP1_2 (STEP)
