File: grbl_board/spinlde_cntrl.sch (KiCad schematic (older format))
At the start: 0 parts

Commit message: spindle control stage (not complete)
Parts:
- added C? (x4): 100n, symbol Device:C
- added J?: 24V_VFD, symbol Connector:Screw_Terminal_01x02
- added R? (x4): 10k, symbol Device:R
- added U?: LMV321, symbol Amplifier_Operational:LMV321
- added U?: 6N137, Package_DIP:DIP-8_W7.62mm, symbol Isolator:6N137
Connections:
- net labels added: 5V, GND, SPINLDE_PWM
- wire segments 0 -> 32
