File: grbl_board/spinlde_cntrl.sch (KiCad schematic (older format))
At the start: 58 parts, among them J14 24V_VFD, J15 Spindle, J16 freq, Q1 BSS127S, Q2 BSS127S, Q3 ZVN4306GTA, Q4 IRF9Z24SPBF, U18 6N137, U19 6N137, U20 6N137, U21 BD9G341EFJ, U22 LMV358, U23 OPA2192, U24 L7805

Commit message: updated README
Parts:
- C31, C32: Digikey Part No. CL05C221JB5NNNC -> 1276-1059-1-ND
Changed lines of the file:
@@
 F 2 "Capacitor_SMD:C_0402_1005Metric_Pad0.74x0.62mm_HandSolder" H 8638 3300 50  0001 C CNN
 F 3 "http://www.samsungsem.com/kr/support/product-search/mlcc/CL05C221JB5NNNC.jsp" H 8600 3450 50  0001 C CNN
-F 4 "CL05C221JB5NNNC" H 8600 3450 50  0001 C CNN "Digikey Part No."
+F 4 "1276-1059-1-ND" H 8600 3450 50  0001 C CNN "Digikey Part No."
 	1    8600 3450
 	1    0    0    -1
@@
 F 2 "Capacitor_SMD:C_0402_1005Metric_Pad0.74x0.62mm_HandSolder" H 8638 4100 50  0001 C CNN
 F 3 "http://www.samsungsem.com/kr/support/product-search/mlcc/CL05C221JB5NNNC.jsp" H 8600 4250 50  0001 C CNN
-F 4 "CL05C221JB5NNNC" H 8600 4250 50  0001 C CNN "Digikey Part No."
+F 4 "1276-1059-1-ND" H 8600 4250 50  0001 C CNN "Digikey Part No."
 	1    8600 4250
 	1    0    0    -1
