File: grbl_board/grbl_controller.sch (KiCad schematic (older format))
At the start: 5 parts

Commit message: finished GRBL controller
Parts:
- added C? (x8): 100n, symbol Device:C
- added C?: 4.7u, symbol Device:C
- added C? (x2): 47p, symbol Device:C
- added D? (x2): LED, symbol Device:LED
- added FB?: Ferrite_Bead, symbol Device:Ferrite_Bead
- added J?: ICSP, symbol Connector_Generic:Conn_02x03_Odd_Even
- added J?: USB_B, symbol Connector:USB_B
- added L?: 10u, symbol Device:L
- added R?: 1M, symbol Device:R
- added R?: 10k, symbol Device:R
- added R? (x2): 27, symbol Device:R
- added R? (x2): 270, symbol Device:R
- added R? (x2): 100, symbol Device:R
- added SW?: SW_Push, symbol Switch:SW_Push_Dual
- added U?: FT231XS, Package_SO:SSOP-20_3.9x8.7mm_P0.635mm, symbol Interface_USB:FT231XS
Connections:
- net GND: now also U?.11 (GND), U?.32 (GND), U?.62 (GND), U?.81 (GND), U?.99 (GND), C?.1, C?.2, C?.2, C?.2, C?.2, C?.2, C?.2, C?.2, C?.2, C?.2, J?.4 (GND), J?.6 (Pin_6), R?.1, R?.2, SW?.2, U?.16 (GND), U?.6 (GND)
- net +5V: now reaches U?.10 (VCC), U?.31 (VCC), U?.61 (VCC), U?.80 (VCC)
- net +5V: now also C?.1, C?.1, C?.1, C?.1, J?.2 (Pin_2), L?.1, R?.1
- net AVCC: now reaches U?.100 (AVCC)
- net AVCC: now also C?.1, L?.2
- net SPINDLE_EN: now reaches U?.15 (PH3)
- net SPINDLE_PWM: now reaches U?.16 (PH4)
- net COOL_FLOOD: now reaches U?.17 (PH5)
- net COOL_MIST: now reaches U?.18 (PH6)
- net RX0: now reaches U?.2 (PE0)
- net RX0: now also R?.1
- net SCK: now reaches U?.20 (PB1)
- net SCK: now also J?.3 (Pin_3)
- net MOSI: now reaches U?.21 (PB2)
- net MOSI: now also J?.4 (Pin_4)
- net MISO: now reaches U?.22 (PB3)
- net MISO: now also J?.1 (Pin_1)
- net LIM_X: now reaches U?.23 (PB4)
- net LIM_Y: now reaches U?.24 (PB5)
- net LIM_Z: now reaches U?.25 (PB6)
- net STEPPER_EN: now reaches U?.26 (PB7)
- net TX0: now reaches U?.3 (PE1)
- net TX0: now also R?.1
- net RESET: now reaches U?.30 (~RESET)
- net RESET: now also C?.1, J?.5 (Pin_5), R?.2, SW?.1
- net SPINDLE_DIR: now reaches U?.5 (PE3)
- net DIR_Z: now reaches U?.58 (PC5)
- net DIR_Y: now reaches U?.59 (PC6)
- net DIR_X: now reaches U?.60 (PC7)
- net STEP_Z: now reaches U?.74 (PA4)
- net STEP_Y: now reaches U?.75 (PA3)
- net STEP_X: now reaches U?.76 (PA2)
- net PROBE: now reaches U?.82 (PK7)
- net DOOR_SAFETY: now reaches U?.86 (PK3)
- net START: now reaches U?.87 (PK2)
- net HOLD: now reaches U?.88 (PK1)
- net RSTABRT: now reaches U?.89 (PK0)
- new net: D?.1 (K), U?.10 (CBUS2)
- new net: C?.1, R?.2, U?.11 (USBDP)
- new net: C?.1, R?.2, U?.12 (USBDM)
- new net: C?.2, U?.13 (3V3OUT), U?.14 (~RESET), U?.3 (VCCIO)
- new net: D?.1 (K), U?.17 (CBUS1)
- new net: R?.2, U?.20 (TXD)
- new net: R?.2, U?.4 (RXD)
- new net: FB?.2, J?.1 (VBUS)
- new net: J?.2 (D-), R?.1
- new net: J?.3 (D+), R?.1
- new net: D?.2 (A), R?.1 (x2)
- new net DTR: C?.2, U?.1 (~DTR)
- new net USBVCC: C?.1, C?.1, FB?.1, R?.2, R?.2, U?.15 (VCC)
Other:
- moved on the sheet: C?, U?, Y?

Commit message: changed to matched resistor
Parts:
- J?: symbol Connector:USB_B -> grbl_board-rescue:USB_B-Connector
Changed lines of the file:
@@
 $EndComp
 $Comp
-L Connector:USB_B J?
+L grbl_board-rescue:USB_B-Connector J?
 U 1 1 61809DB5
 P 1350 4000
