File: grbl_board/grbl_controller.sch (KiCad schematic (older format))
At the start: 32 parts

Commit message: added some footprint associations
Parts:
- removed SW?: SW_Push, symbol Switch:SW_Push_Dual
- added SW1: SW_Push, Button_Switch_SMD:SW_Push_1P1T_NO_6x6mm_H9.5mm, symbol Switch:SW_Push
- C1: renamed from C?; footprint (none) -> Capacitor_SMD:C_1206_3216Metric_Pad1.33x1.80mm_HandSolder; Digikey Part No. (none) -> 1276-6781-1-ND
- C10, C11, C12, C13, C14, C3, C5, C8, C9: renamed from C?; footprint (none) -> Capacitor_SMD:C_0603_1608Metric_Pad1.05x0.95mm_HandSolder; Digikey Part No. (none) -> 1276-1941-1-ND
- C2, C4: renamed from C?; footprint (none) -> Capacitor_SMD:C_0402_1005Metric_Pad0.74x0.62mm_HandSolder; Digikey Part No. (none) -> 1276-1699-1-ND
- C6, C7: renamed from C?; footprint (none) -> Capacitor_SMD:C_0603_1608Metric_Pad1.05x0.95mm_HandSolder; Digikey Part No. (none) -> 1276-1187-1-ND
- FB1: renamed from FB?; footprint (none) -> Capacitor_SMD:C_0603_1608Metric_Pad1.05x0.95mm_HandSolder; Digikey Part No. (none) -> 732-1591-1-ND
- J3: renamed from J?; footprint (none) -> Connector_USB:USB_B_OST_USB-B1HSxx_Horizontal; Digikey Part No. (none) -> 380-1492-ND
- J4: renamed from J?; footprint (none) -> Connector_PinHeader_2.54mm:PinHeader_2x03_P2.54mm_Vertical; Digikey Part No. (none) -> 609-3234-ND
- L1: renamed from L?; footprint (none) -> Inductor_SMD:L_0805_2012Metric_Pad1.05x1.20mm_HandSolder; Digikey Part No. (none) -> 490-4029-1-ND
- R1, R2: renamed from R?; footprint (none) -> Resistor_SMD:R_0603_1608Metric_Pad0.98x0.95mm_HandSolder; Digikey Part No. (none) -> 311-27GRCT-ND
- R3: renamed from R?; footprint (none) -> Resistor_SMD:R_0603_1608Metric_Pad0.98x0.95mm_HandSolder; Digikey Part No. (none) -> 311-1.0MGRCT-ND
- R4, R7: renamed from R?; footprint (none) -> Resistor_SMD:R_0805_2012Metric_Pad1.15x1.40mm_HandSolder; Digikey Part No. (none) -> YAG6172CT-ND
- R5, R6: renamed from R?; footprint (none) -> Resistor_SMD:R_0603_1608Metric_Pad0.98x0.95mm_HandSolder; Digikey Part No. (none) -> 311-100GRCT-ND
- R8: renamed from R?; footprint (none) -> Resistor_SMD:R_0805_2012Metric_Pad1.15x1.40mm_HandSolder; Digikey Part No. (none) -> 311-10KARCT-ND
- U1: renamed from U?; Digikey Part No. (none) -> 768-1129-1-ND
- Y1: renamed from Y?; footprint (none) -> Crystal:Crystal_SMD_SeikoEpson_TSX3225-4Pin_3.2x2.5mm_HandSoldering; Digikey Part No. (none) -> SER4372CT-ND
- gave numbers to parts that had none: 3
